File: kicad/pxref25.kicad_pcb (KiCad board)
At the start: 2 copper layers, 48.9 x 46.4 mm, 57 parts, among them P1 CONN_1X1, P2 CONN_1X1, P3 CONN_1X1, P4 CONN_1X1, P5 CONN_1X1, Q1 2N3904, U1 LTZ1000A, U2 LT1013, U30 LTC2057

Commit message: branching files for 2.5.x
Parts:
- added H***: Val**, hole_M3, F.Cu at (188.0, 71.8)
- added H***: Val**, hole_M3, F.Cu at (257.2, 109.2)
- added H***: Val**, 1pin_032_058, F.Cu at (215.3, 75.6)
- added H***: Val**, 1pin_032_058, F.Cu at (220.3, 75.6)
- added H***: Val**, 1pin_032_058, F.Cu at (224.8, 80.0)
- added H***: Val**, 1pin_032_058, F.Cu at (224.8, 85.1)
- added H***: Val**, 1pin_032_058, F.Cu at (210.8, 80.0)
- added H***: Val**, 1pin_032_058, F.Cu at (210.8, 85.1)
- added H***: Val**, 1pin_032_058, F.Cu at (215.3, 89.5)
- added H***: Val**, 1pin_032_058, F.Cu at (220.3, 89.5)
- added ferrite_core_20x12_PL: VAL**, ferrite_core_20x12_PL, F.Cu at (254.6, 92.1)
- added ferrite_core_20x12_PL: VAL**, ferrite_core_20x12_PL, F.Cu at (191.1, 90.2)
- moved H*** 14.6 mm to (257.2, 71.8)
- moved H1 14.6 mm to (188.0, 109.2)
Other:
- board size 48.9 x 46.4 mm -> 78.1 x 46.4 mm
