File: kicad/pxref26.kicad_pcb (KiCad board)
At the start: 2 copper layers, 78.1 x 46.4 mm, 71 parts, among them P1 CONN_2X1, P2 CONN_1X1, P3 CONN_1X1, P5 CONN_1X1, P6 CONN_2X1, Q1 2N3904, U1 LTZ1000A, U2 LT1013, U30 LTC2057

Commit message: v2.6
Parts:
- removed C41: 10uF, ELCAP_10_20_V_059A
- removed C9: 0.1uF, BOXCAP_01_03_02_059A
- removed the G*** at (196.8, 71.5)
- removed R2, R3: 70k, R_BOX_HERMETIC_PL
- removed R4: 13k, R_BOX_PL
- removed R45: 13k/1k, R_BOX_DIVIDER_PL
- removed R5: 1k, R_BOX_PL
- added G***: OSHW-logo_silkscreen-front_4mm, OSHW-logo_silkscreen-front_4mm, F.Cu at (190.5, 102.2)
- added JP3: JUMPER2, SIL-2, F.Cu at (213.4, 104.8)
- added JP5: JUMPER2, SIL-2, F.Cu at (210.8, 107.3)
- added JP50: JUMPER2, SIL-2, F.Cu at (198.1, 103.5)
- added JP51: JUMPER2, SIL-2, F.Cu at (210.8, 102.2)
- added JP52: JUMPER2, SIL-2, F.Cu at (195.6, 106.0)
- added JP54: JUMPER2, SIL-2, F.Cu at (198.1, 108.6)
- added JP56: JUMPER2, SIL-2, F.Cu at (195.6, 111.1)
- added R50: OHMTEK_132077, DIP16_PL, F.Cu at (200.7, 94.0)
- R1: footprint R_BOX_HERMETIC_PL -> R_BOX_HERMETIC_WW_AXIAL_07_PL
- moved R40 44.2 mm to (202.6, 68.6), turned to 180 degrees
- moved D4 42.0 mm to (185.4, 97.2), turned to 270 degrees
- moved L40 41.9 mm to (193.7, 70.5), turned to 0 degrees
- moved C40 38.1 mm to (208.9, 71.1), turned to 270 degrees
- moved R9 19.3 mm to (231.1, 77.5), turned to 270 degrees
- moved R19 13.2 mm to (224.8, 111.1)
- moved R31 9.61 mm to (233.7, 77.5), turned to 270 degrees
- moved P1 2.68 mm to (193.0, 88.3)
- moved C11 2.01 mm to (211.5, 91.4)
- moved R30 1.80 mm to (229.2, 74.9)
- moved C12 1.27 mm to (207.6, 82.5)
- moved R1 0.90 mm to (202.6, 81.9)
Connections:
- net N-0000016 renamed R2L
- net N-000005 renamed R4L
- net Vz+ Sense renamed R2H
- net Vz- Sense renamed R5L
- C14 pad 2: N-0000024 (its old number) -> R3L
- C2 pad 1: N-0000024 (its old number) -> R3L
- U1 pad 8: N-0000024 (its old number) -> R3L
- U2 pad 3: N-0000024 (its old number) -> R3L
Routing:
- net 15V: track 52.1 -> 101.2 mm
- net R3L: track 0.00 -> 45.1 mm, vias 0 -> 2
- net N-0000024 (its old number): track 36.9 -> 0.00 mm, vias 1 -> 0
- net N-0000028: track 55.3 -> 90.6 mm, vias 1 -> 3
- net R2H: track 127.8 -> 100.7 mm
- net N-000003: track 33.9 -> 13.5 mm
- net H+: track 76.9 -> 57.6 mm
- net R4L: track 32.7 -> 49.2 mm
- net N-000004: track 23.4 -> 38.9 mm
- net R5L: track 354.9 -> 342.2 mm
- net N-0000030: track 19.6 -> 8.67 mm
- net Vz+ Buf: track 50.2 -> 39.7 mm
- net N-000001: track 10.5 -> 2.29 mm
- net R2L: track 52.7 -> 59.0 mm
- net N-0000017: track 0.00 -> 5.71 mm
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Other:
- outline, holes or cut-outs redrawn
- board text added: "v2.6"
- board text removed: "v2.5"
